File: atreus-butterfly-62.sch (KiCad schematic (older format))
At the start: 76 parts, among them J1 USB_OTG, J2 Conn_01x04, SW1 SW_Push, SW10 SW_Push, SW11 SW_Push, SW12 SW_Push, SW13 SW_Push, SW14 SW_Push, SW15 SW_Push, SW16 SW_Push, SW17 SW_Push, SW18 SW_Push, SW19 SW_Push, SW2 SW_Push, SW20 SW_Push, SW21 SW_Push, SW22 SW_Push, SW23 SW_Push, SW24 SW_Push, SW25 SW_Push, SW26 SW_Push, SW27 SW_Push, SW28 SW_Push, SW29 SW_Push, SW3 SW_Push, SW30 SW_Push, SW31 SW_Push, SW32 SW_Push, SW4 SW_Push, SW5 SW_Push, SW6 SW_Push, SW7 SW_Push, SW8 SW_Push, SW9 SW_Push, U1 ATMEGA32U4-MU, Y1 Crystal

Commit message: more stuff done no idea really
Parts:
- C1, C2, C3, C4: symbol device:C_Small -> atreus-butterfly-62-rescue:C_Small-device
- D1, D10, D11, D12, D13, D14, D15, D16, D17, D18, D19, D2, D20, D21, D22, D23, D24, D25, D26, D27, D28, D29, D3, D30, D31, D32, D4, D5, D6, D7, D8, D9: symbol device:D -> atreus-butterfly-62-rescue:D-device
- R1, R2, R3, R4: symbol device:R_Small -> atreus-butterfly-62-rescue:R_Small-device
- SW1, SW10, SW11, SW12, SW13, SW14, SW15, SW16, SW17, SW18, SW19, SW2, SW20, SW21, SW22, SW23, SW24, SW25, SW26, SW27, SW28, SW29, SW3, SW30, SW31, SW32, SW4, SW5, SW6, SW7, SW8, SW9: footprint ourglass_v7:Kailh_low_profile -> kailh:Kailh_low_profile
- Y1: symbol device:Crystal -> atreus-butterfly-62-rescue:Crystal-device
